File: hardware/PULSAR.kicad_sch (KiCad schematic)
At the start: 3 parts, among them U1 AP2112K-3.3

Commit message: feat: add Hall sensor SS49E schematic with HALL_OUT_1 net
Parts:
- added U2: SS49E, symbol Connector_Generic:Conn_01x03
Connections:
- net +3.3V: now also U2.1 (Pin_1)
- net GND: now also U2.2 (Pin_2)
- new net HALL_OUT_1: U2.3 (Pin_3)
